Commit message: Add approximate RobotDigg TCP and finger frames
Co-authored-by: Stanisław Piasecki <Stachq1@users.noreply.github.com>

File: fairino_description/urdf/FR3WML.urdf (robot description, URDF)
Before this commit: robot FR3WML, 8 links, 7 joints
Links:
- added link robotdigg_left_finger; collision box size=0.025 0.012 0.100; visual box size=0.025 0.012 0.100
- added link robotdigg_right_finger; collision box size=0.025 0.012 0.100; visual box size=0.025 0.012 0.100
- added link robotdigg_tcp
Joints:
- added joint robotdigg_left_finger_joint: type fixed, parent flange_Link, child robotdigg_left_finger, origin xyz=0 0.036 0.130 rpy=0 0 0
- added joint robotdigg_right_finger_joint: type fixed, parent flange_Link, child robotdigg_right_finger, origin xyz=0 -0.036 0.130 rpy=0 0 0
- added joint robotdigg_tcp_joint: type fixed, parent flange_Link, child robotdigg_tcp, origin xyz=0 0 0.130 rpy=0 0 0

Commit message: Refine RobotDigg gripper geometry
Co-authored-by: Stanisław Piasecki <Stachq1@users.noreply.github.com>

File: fairino_description/urdf/FR3WML.urdf (robot description, URDF)
Before this commit: robot FR3WML, 11 links, 10 joints
Links:
- added link robotdigg_gripper_base; collision box size=0.080 0.110 0.068; visual box size=0.080 0.110 0.068
- link robotdigg_left_finger: geometry collision box size=0.025 0.012 0.140; visual box size=0.025 0.012 0.140
- link robotdigg_right_finger: geometry collision box size=0.025 0.012 0.140; visual box size=0.025 0.012 0.140
Joints:
- added joint robotdigg_gripper_base_joint: type fixed, parent flange_Link, child robotdigg_gripper_base, origin xyz=0 0 0.034 rpy=0 0 0
- joint robotdigg_left_finger_joint: origin xyz=0 0.036 0.130 rpy=0 0 0 -> xyz=0 0.035 0.140 rpy=0.139626 0 0
- joint robotdigg_right_finger_joint: origin xyz=0 -0.036 0.130 rpy=0 0 0 -> xyz=0 -0.035 0.140 rpy=-0.139626 0 0
- joint robotdigg_tcp_joint: origin xyz=0 0 0.130 rpy=0 0 0 -> xyz=0 0 0.140 rpy=0 0 0

Commit message: Set open gripper pose and flange twist
Co-authored-by: Stanisław Piasecki <Stachq1@users.noreply.github.com>

File: fairino_description/urdf/FR3WML.urdf (robot description, URDF)
Before this commit: robot FR3WML, 12 links, 11 joints
Links:
- link robotdigg_gripper_base: geometry collision box size=0.080 0.120 0.068; visual box size=0.080 0.120 0.068
- link robotdigg_left_finger: geometry collision box size=0.025 0.012 0.119; visual box size=0.025 0.012 0.119
- link robotdigg_right_finger: geometry collision box size=0.025 0.012 0.119; visual box size=0.025 0.012 0.119
Joints:
- joint robotdigg_gripper_base_joint: origin xyz=0 0 0.034 rpy=0 0 0 -> xyz=0 0 0.034 rpy=0 0 0.785398
- joint robotdigg_left_finger_joint: origin xyz=0 0.035 0.140 rpy=0.139626 0 0 -> xyz=0 0.045 0.106 rpy=0.139626 0 0; parent flange_Link -> robotdigg_gripper_base
- joint robotdigg_right_finger_joint: origin xyz=0 -0.035 0.140 rpy=-0.139626 0 0 -> xyz=0 -0.045 0.106 rpy=-0.139626 0 0; parent flange_Link -> robotdigg_gripper_base
- joint robotdigg_tcp_joint: origin xyz=0 0 0.140 rpy=0 0 0 -> xyz=0 0 0.106 rpy=0 0 0; parent flange_Link -> robotdigg_gripper_base

Commit message: Correct open gripper V geometry
Co-authored-by: Stanisław Piasecki <Stachq1@users.noreply.github.com>

File: fairino_description/urdf/FR3WML.urdf (robot description, URDF)
Before this commit: robot FR3WML, 12 links, 11 joints
Links:
- link robotdigg_gripper_base: geometry collision box size=0.070 0.090 0.060; visual box size=0.070 0.090 0.060
Joints:
- joint robotdigg_gripper_base_joint: origin xyz=0 0 0.034 rpy=0 0 0.785398 -> xyz=0 0 0.030 rpy=0 0 0.785398
- joint robotdigg_left_finger_joint: origin xyz=0 0.045 0.106 rpy=0.139626 0 0 -> xyz=0 0.0556509 0.110 rpy=-0.342810 0 0
- joint robotdigg_right_finger_joint: origin xyz=0 -0.045 0.106 rpy=-0.139626 0 0 -> xyz=0 -0.0556509 0.110 rpy=0.342810 0 0
- joint robotdigg_tcp_joint: origin xyz=0 0 0.106 rpy=0 0 0 -> xyz=0 0 0.110 rpy=0 0 0

Commit message: Shorten fingers and close palm clearance
Co-authored-by: Stanisław Piasecki <Stachq1@users.noreply.github.com>

File: fairino_description/urdf/FR3WML.urdf (robot description, URDF)
Before this commit: robot FR3WML, 12 links, 11 joints
Links:
- link robotdigg_gripper_base: geometry collision box size=0.070 0.090 0.084; visual box size=0.070 0.090 0.084
- link robotdigg_left_finger: geometry collision box size=0.025 0.012 0.109; visual box size=0.025 0.012 0.109
- link robotdigg_right_finger: geometry collision box size=0.025 0.012 0.109; visual box size=0.025 0.012 0.109
Joints:
- joint robotdigg_gripper_base_joint: origin xyz=0 0 0.030 rpy=0 0 0.785398 -> xyz=0 0 0.042 rpy=0 0 0.785398
- joint robotdigg_left_finger_joint: origin xyz=0 0.0556509 0.110 rpy=-0.342810 0 0 -> xyz=0 0.0555814 0.098 rpy=-0.375752 0 0
- joint robotdigg_right_finger_joint: origin xyz=0 -0.0556509 0.110 rpy=0.342810 0 0 -> xyz=0 -0.0555814 0.098 rpy=0.375752 0 0
- joint robotdigg_tcp_joint: origin xyz=0 0 0.110 rpy=0 0 0 -> xyz=0 0 0.098 rpy=0 0 0
